Commit message: All files in place

File: my_robot/urdf/my_robot.xacro (robot description, xacro)
@@ -150,4 +150,13 @@
 	<axis xyz="0 1 0" rpy="0 0 0"/>
 </joint>
+<!-- OPTICAL CAMERA -->
+  <joint name="camera_optical_joint" type="fixed">
+    <origin xyz="0 0 0" rpy="-1.5707 0 -1.5707"/>
+    <parent link="camera"/>
+    <child link="camera_link_optical"/>
+  </joint>
+  <link name="camera_link_optical">
+  </link>
+<!---->
 <link name='hokuyo'>
 	<pose> 0 0 0 0 0 0 </pose>
